Commit message: Building of reacher_env Stuck at torque control

File: assets/ur5/model.urdf (robot description, URDF)
Before this commit: robot universal_robot, 7 links, 6 joints
Joints:
- joint shoulder_lift_joint: limit lower=-6.28318530718 upper=6.28318530718 effort=150.0 velocity=3.15 -> lower=0 upper=3.14159 effort=150.0 velocity=3.15

File: assets/ur5_w_gripper/model.urdf (robot description, URDF)
Before this commit: robot universal_robot, 18 links, 17 joints
Joints:
- joint shoulder_lift_joint: limit lower=-6.28318530718 upper=6.28318530718 effort=150.0 velocity=3.15 -> lower=-3.14159 upper=0 effort=150.0 velocity=3.15
