Commit message: updated model removed plane

File: assets/ur5_w_gripper/model.urdf (robot description, URDF)
Before this commit: robot universal_robot, 18 links, 17 joints
Joints:
- joint shoulder_lift_joint: limit lower=-3.14159 upper=0 effort=150.0 velocity=3.15 -> lower=-3.14159 upper=3.14159 effort=150.0 velocity=3.15

Commit message: added limit for joint and goal

File: assets/ur5_w_gripper/model.urdf (robot description, URDF)
Before this commit: robot universal_robot, 18 links, 17 joints
Links:
- removed link bh_base_link
- removed link bh_finger_11_link
- removed link bh_finger_12_link
- removed link bh_finger_13_link
- removed link bh_finger_21_link
- removed link bh_finger_22_link
- removed link bh_finger_23_link
- removed link bh_finger_31_link
- removed link bh_finger_32_link
- removed link bh_finger_33_link
- link ee_link: mass None -> 0.
Joints:
- removed joint arm_gripper_joint
- removed joint bh_j11_joint
- removed joint bh_j12_joint
- removed joint bh_j13_joint
- removed joint bh_j21_joint
- removed joint bh_j22_joint
- removed joint bh_j23_joint
- removed joint bh_j31_joint
- removed joint bh_j32_joint
- removed joint bh_j33_joint
- joint elbow_joint: limit lower=-3.14159265359 upper=3.14159265359 effort=150.0 velocity=3.15 -> lower=-1.57 upper=2.5 effort=150.0 velocity=3.15
- joint shoulder_lift_joint: limit lower=-3.14159 upper=3.14159 effort=150.0 velocity=3.15 -> lower=-1.57 upper=0 effort=150.0 velocity=3.15
- joint shoulder_pan_joint: limit lower=-6.28318530718 upper=6.28318530718 effort=150.0 velocity=3.15 -> lower=-0.785 upper=0.785 effort=150.0 velocity=3.15
- joint wrist_1_joint: limit lower=-6.28318530718 upper=6.28318530718 effort=28.0 velocity=3.2 -> lower=-3.1415 upper=3.1415 effort=28.0 velocity=13.2
- joint wrist_2_joint: limit lower=-6.28318530718 upper=6.28318530718 effort=28.0 velocity=3.2 -> lower=-3.1415 upper=3.1415 effort=28.0 velocity=13.2
- joint wrist_3_joint: limit lower=-6.28318530718 upper=6.28318530718 effort=28.0 velocity=3.2 -> lower=-3.1415 upper=3.1415 effort=28.0 velocity=13.2

Commit message: final working on lab com

File: assets/ur5_w_gripper/model.urdf (robot description, URDF)
Before this commit: robot universal_robot, 8 links, 7 joints
Joints:
- joint shoulder_lift_joint: limit lower=-1.57 upper=0 effort=150.0 velocity=3.15 -> lower=-1.57 upper=1.57 effort=150.0 velocity=3.15
