Commit message: updated robot model and reward dist calculation

File: assets/ur5_w_gripper/3f_2j.urdf (robot description, URDF)
Before this commit: robot ur5_2f1j, 24 links, 23 joints
Links:
- link f11_base: mass None -> 0.01
- link f12_slot: mass None -> 0.01
- link f13_slot: mass None -> 0.
- link f21_base: mass None -> 0.01
- link f22_slot: mass None -> 0.01
- link f23_slot: mass None -> 0.
- link f31_base: mass None -> 0.
- link f32_slot: mass None -> 0.
- link f33_slot: mass None -> 0.
Joints:
- joint ee_fixed_joint: origin xyz=0.0 0.0823. 0. rpy=0.0 0.0 1.57079632679 -> xyz=0.0 0.0823 0.0 rpy=0.0 0.0 1.57079632679
- joint f12_joint: origin xyz=0 0 .0 rpy=0 -.0 0 -> xyz=0 0 0.0 rpy=0 -0.0 0
- joint f12_slot_joint: origin xyz=0 0 .05 rpy=0 0 0 -> xyz=0 0 0.05 rpy=0 0 0
- joint f21_joint: origin xyz=0 0 .0 rpy=.25 -.25 0 -> xyz=0 0 0.0 rpy=.25 -0.25 0
- joint f31_joint: origin xyz=0 .0 .0 rpy=-.25 -.25 0 -> xyz=0 0.0 0.0 rpy=-0.25 -0.25 0
- joint f32_joint: origin xyz=0 0 .0 rpy=0 -.0 0 -> xyz=0. 0. .0 rpy=0 .0 0
- joint f32_slot_joint: origin xyz=0 0 .05 rpy=0 0 0 -> xyz=0 0 0.05 rpy=0 0 0
- joint f33_slot_joint: origin xyz=0 0 .05 rpy=0 0 0 -> xyz=0 0 0.05 rpy=0 0 0
