Commit message: added lib for MULTI_ROBOT HCP

File: assets/ur5_w_gripper/2f_1j.urdf (robot description, URDF)
Before this commit: robot ur5_2f1j, 15 links, 14 joints
Joints:
- joint ee_fixed_joint: origin xyz=0.0 0.0823. 0. rpy=0.0 0.0 1.57079632679 -> xyz=0.0 0.0823 0.0 rpy=0.0 0.0 1.57079632679
- joint f11_base_joint: origin xyz=.05 0 .0 rpy=0 0 0 -> xyz=0.05 0 .0 rpy=0 0 0
- joint f11_joint: origin xyz=0 0 .0 rpy=0 .25 0 -> xyz=0 0 .0 rpy=0 0.25 0
- joint f12_slot_joint: origin xyz=0 0 .1 rpy=0 0 0 -> xyz=0 0 0.1 rpy=0 0 0
- joint f21_base_joint: origin xyz=-.05 -0.0 .0 rpy=0 0 0 -> xyz=-0.05 -0.0 0.0 rpy=0 0 0
- joint f21_joint: origin xyz=0 0 .0 rpy=.0 -.25 0 -> xyz=0 0 .0 rpy=0.0 -0.25 0
- joint f22_slot_joint: origin xyz=0 0 .1 rpy=0 0 0 -> xyz=0 0 0.1 rpy=0 0 0

File: assets/ur5_w_gripper/2f_2j.urdf (robot description, URDF)
Before this commit: robot ur5_2f2j, 19 links, 18 joints
Joints:
- joint ee_fixed_joint: origin xyz=0.0 0.0823. 0. rpy=0.0 0.0 1.57079632679 -> xyz=0.0 0.0823 0. rpy=0.0 0.0 1.57079632679

File: assets/ur5_w_gripper/3f_1j.urdf (robot description, URDF)
Before this commit: robot ur5_3f1j, 21 links, 20 joints
Links:
- removed link f12
- removed link f22
- removed link f32
- link f11: geometry collision cylinder length=.1 radius=.01; visual cylinder length=.1 radius=.01
- link f21: geometry collision cylinder length=.1 radius=.01; visual cylinder length=.1 radius=.01
- link f31: geometry collision cylinder length=.1 radius=.01; visual cylinder length=.1 radius=.01
Joints:
- removed joint f12_joint
- removed joint f22_joint
- removed joint f32_joint
- joint ee_fixed_joint: origin xyz=0.0 0.0823. 0. rpy=0.0 0.0 1.57079632679 -> xyz=0.0 0.0823 0.0 rpy=0.0 0.0 1.57079632679
- joint f11_joint: limit lower=-.4 upper=.25 effort=30 velocity=2.0 -> lower=-.65 upper=.25 effort=30 velocity=2.0
- joint f12_slot_joint: origin xyz=0 0 .05 rpy=0 0 0 -> xyz=0 0 .1 rpy=0 0 0
- joint f21_joint: limit lower=-.4 upper=.25 effort=30 velocity=2.0 -> lower=-.65 upper=.25 effort=30 velocity=2.0; mimic (none) -> joint=f11_joint multiplier=1
- joint f22_slot_joint: origin xyz=0 0 .05 rpy=0 0 0 -> xyz=0 0 .1 rpy=0 0 0
- joint f31_joint: limit lower=-.4 upper=.25 effort=30 velocity=2.0 -> lower=-.65 upper=.25 effort=30 velocity=2.0; mimic (none) -> joint=f11_joint multiplier=1
- joint f32_slot_joint: origin xyz=0 0 .05 rpy=0 0 0 -> xyz=0 0 .1 rpy=0 0 0
- joint palm_ee_joint: origin xyz=0.0 0. 0. rpy=3.14 1.57 3.14 -> xyz=0.0 0.0 0.0 rpy=3.14 1.57 3.14
