Commit message: complete custom gripper model

File: assets/grippers/2f_1j.urdf (robot description, URDF)
Before this commit: robot gripper_3f_1j, 7 links, 6 joints
Links:
- removed link finger_3
- removed link finger_3_slot
Joints:
- removed joint finger_3_joint
- removed joint finger_3_slot_joint
- joint finger_2_joint: axis 1 -1 0 ->  -1 0; origin xyz=0 0 .0 rpy=.25 -.25 0 -> xyz=0 0 .0 rpy=0 -.25 0
- joint finger_2_slot_joint: origin xyz=-.025 -0.043301270189222 .0 rpy=0 0 0 -> xyz=-.05 0 .0 rpy=0 0 0

File: assets/grippers/2f_2j.urdf (robot description, URDF)
Before this commit: robot gripper_3f_1j, 7 links, 6 joints
Links:
- removed link finger_1
- removed link finger_1_slot
- removed link finger_2
- removed link finger_2_slot
- removed link finger_3
- removed link finger_3_slot
- added link f11; collision cylinder length=.05 radius=.01; visual cylinder length=.05 radius=.01
- added link f11_slot; visual sphere radius=.015
- added link f12; collision cylinder length=.05 radius=.01; visual cylinder length=.05 radius=.01
- added link f12_slot; visual sphere radius=.015
- added link f21; collision cylinder length=.05 radius=.01; visual cylinder length=.05 radius=.01
- added link f21_slot; visual sphere radius=.015
- added link f22; collision cylinder length=.05 radius=.01; visual cylinder length=.05 radius=.01
- added link f22_slot; visual sphere radius=.015
Joints:
- removed joint finger_1_joint
- removed joint finger_1_slot_joint
- removed joint finger_2_joint
- removed joint finger_2_slot_joint
- removed joint finger_3_joint
- removed joint finger_3_slot_joint
- added joint f11_joint: type revolute, parent f11_slot, child f11, origin xyz=0 0 .0 rpy=0 .25 0, axis 0 1 0, limit lower=-.4 upper=.25 effort=30 velocity=2.0
- added joint f11_slot_joint: type fixed, parent palm, child f11_slot, origin xyz=.05 0 .0 rpy=0 0 0
- added joint f12_joint: type revolute, parent f12_slot, child f12, origin xyz=0 0 .0 rpy=0 -.0 0, axis 0 1 0, limit lower=-.65 upper=.0 effort=30 velocity=2.0, mimic joint=f11_joint multiplier=1 offset=-.25
- added joint f12_slot_joint: type fixed, parent f11, child f12_slot, origin xyz=0 0 .05 rpy=0 0 0
- added joint f21_joint: type revolute, parent f21_slot, child f21, origin xyz=0 0 .0 rpy=.0 -.25 0, axis 0 -1 0, limit lower=-.4 upper=.25 effort=30 velocity=2.0
- added joint f21_slot_joint: type fixed, parent palm, child f21_slot, origin xyz=-.05 -0.0 .0 rpy=0 0 0
- added joint f22_joint: type revolute, parent f22_slot, child f22, origin xyz=0 0 .0 rpy=0 -.0 0, axis 0 -1 0, limit lower=-.65 upper=.0 effort=30 velocity=2.0, mimic joint=f21_joint multiplier=1 offset=-.25
- added joint f22_slot_joint: type fixed, parent f21, child f22_slot, origin xyz=0 0 .05 rpy=0 0 0

Commit message: motion of fingers configured

File: assets/grippers/2f_1j.urdf (robot description, URDF)
Before this commit: robot gripper_3f_1j, 5 links, 4 joints
Links:
- removed link finger_1
- removed link finger_1_slot
- removed link finger_2
- removed link finger_2_slot
- added link f11; collision cylinder length=.1 radius=.01; visual cylinder length=.1 radius=.01
- added link f11_slot; visual sphere radius=.015
- added link f21; collision cylinder length=.1 radius=.01; visual cylinder length=.1 radius=.01
- added link f21_slot; visual sphere radius=.015
- link palm: geometry collision cylinder length=0.03 radius=0.05; visual cylinder length=0.03 radius=0.05
Joints:
- removed joint finger_1_joint
- removed joint finger_1_slot_joint
- removed joint finger_2_joint
- removed joint finger_2_slot_joint
- added joint f11_joint: type revolute, parent f11_slot, child f11, origin xyz=0 0 .0 rpy=0 .25 0, axis 0 1 0, limit lower=-.6 upper=.25 effort=30 velocity=2.0
- added joint f11_slot_joint: type fixed, parent palm, child f11_slot, origin xyz=.05 0 .0 rpy=0 0 0
- added joint f21_joint: type revolute, parent f21_slot, child f21, origin xyz=0 0 .0 rpy=.0 -.25 0, axis 0 -1 0, limit lower=-.6 upper=.25 effort=30 velocity=2.0
- added joint f21_slot_joint: type fixed, parent palm, child f21_slot, origin xyz=-.05 -0.0 .0 rpy=0 0 0

File: assets/grippers/2f_2j.urdf (robot description, URDF)
Before this commit: robot gripper_3f_1j, 9 links, 8 joints
Links:
- link palm: geometry collision cylinder length=0.03 radius=0.05; visual cylinder length=0.03 radius=0.05

File: assets/grippers/3f_1j.urdf (robot description, URDF)
Before this commit: robot gripper_3f_1j, 7 links, 6 joints
Links:
- link palm: geometry collision cylinder length=0.03 radius=0.05; visual cylinder length=0.03 radius=0.05
Joints:
- joint finger_1_joint: limit lower=-.6 upper=.25 effort=30 velocity=2.0 -> lower=-.65 upper=.25 effort=30 velocity=2.0
- joint finger_2_joint: limit lower=-.6 upper=.25 effort=30 velocity=2.0 -> lower=-.65 upper=.25 effort=30 velocity=2.0
- joint finger_3_joint: limit lower=-.6 upper=.25 effort=30 velocity=2.0 -> lower=-.65 upper=.25 effort=30 velocity=2.0

File: assets/grippers/3f_2j.urdf (robot description, URDF)
Before this commit: robot gripper_3f_1j, 13 links, 12 joints
Links:
- link palm: geometry collision cylinder length=0.03 radius=0.05; visual cylinder length=0.03 radius=0.05

Commit message: added env for gripper with arm

File: assets/grippers/2f_1j.urdf (robot description, URDF)
Before this commit: robot gripper_3f_1j, 5 links, 4 joints
Links:
- removed link f11_slot
- removed link f21_slot
- added link f11_base; visual sphere radius=.015
- added link f21_base; visual sphere radius=.015
Joints:
- removed joint f11_slot_joint
- removed joint f21_slot_joint
- added joint f11_base_joint: type fixed, parent palm, child f11_base, origin xyz=.05 0 .0 rpy=0 0 0
- added joint f21_base_joint: type fixed, parent palm, child f21_base, origin xyz=-.05 -0.0 .0 rpy=0 0 0
- joint f11_joint: parent f11_slot -> f11_base
- joint f21_joint: parent f21_slot -> f21_base

File: assets/grippers/2f_2j.urdf (robot description, URDF)
Before this commit: robot gripper_3f_1j, 9 links, 8 joints
Links:
- removed link f11_slot
- removed link f21_slot
- added link f11_base; visual sphere radius=.015
- added link f21_base; visual sphere radius=.015
Joints:
- removed joint f11_slot_joint
- removed joint f21_slot_joint
- added joint f11_base_joint: type fixed, parent palm, child f11_base, origin xyz=.05 0 .0 rpy=0 0 0
- added joint f21_base_joint: type fixed, parent palm, child f21_base, origin xyz=-.05 -0.0 .0 rpy=0 0 0
- joint f11_joint: parent f11_slot -> f11_base
- joint f21_joint: parent f21_slot -> f21_base

File: assets/grippers/3f_1j.urdf (robot description, URDF)
Before this commit: robot gripper_3f_1j, 7 links, 6 joints
Links:
- removed link finger_1
- removed link finger_1_slot
- removed link finger_2
- removed link finger_2_slot
- removed link finger_3
- removed link finger_3_slot
- added link f11; collision cylinder length=.1 radius=.01; visual cylinder length=.1 radius=.01
- added link f11_base; visual sphere radius=.015
- added link f21; collision cylinder length=.1 radius=.01; visual cylinder length=.1 radius=.01
- added link f21_base; visual sphere radius=.015
- added link f31; collision cylinder length=.1 radius=.01; visual cylinder length=.1 radius=.01
- added link f31_base; visual sphere radius=.015
Joints:
- removed joint finger_1_joint
- removed joint finger_1_slot_joint
- removed joint finger_2_joint
- removed joint finger_2_slot_joint
- removed joint finger_3_joint
- removed joint finger_3_slot_joint
- added joint f11_base_joint: type fixed, parent palm, child f11_base, origin xyz=.05 0 .0 rpy=0 0 0
- added joint f11_joint: type revolute, parent f11_base, child f11, origin xyz=0 0 .0 rpy=0 .25 0, axis 0 1 0, limit lower=-.65 upper=.25 effort=30 velocity=2.0
- added joint f21_base_joint: type fixed, parent palm, child f21_base, origin xyz=-.025 -0.043301270189222 .0 rpy=0 0 0
- added joint f21_joint: type revolute, parent f21_base, child f21, origin xyz=0 0 .0 rpy=.25 -.25 0, axis 1 -1 0, limit lower=-.65 upper=.25 effort=30 velocity=2.0, mimic joint=f11_joint multiplier=1
- added joint f31_base_joint: type fixed, parent palm, child f31_base, origin xyz=-.025 0.043301270189222 .0 rpy=0 0 0
- added joint f31_joint: type revolute, parent f31_base, child f31, origin xyz=0 .0 .0 rpy=-.25 -.25 0, axis -1 -1 0, limit lower=-.65 upper=.25 effort=30 velocity=2.0, mimic joint=f11_joint multiplier=1

File: assets/grippers/3f_2j.urdf (robot description, URDF)
Before this commit: robot gripper_3f_1j, 13 links, 12 joints
Links:
- removed link f11_slot
- removed link f21_slot
- removed link f31_slot
- added link f11_base; visual sphere radius=.015
- added link f21_base; visual sphere radius=.015
- added link f31_base; visual sphere radius=.015
Joints:
- removed joint f11_slot_joint
- removed joint f21_slot_joint
- removed joint f31_slot_joint
- added joint f11_base_joint: type fixed, parent palm, child f11_base, origin xyz=.05 0 .0 rpy=0 0 0
- added joint f21_base_joint: type fixed, parent palm, child f21_base, origin xyz=-.025 -0.043301270189222 .0 rpy=0 0 0
- added joint f31_base_joint: type fixed, parent palm, child f31_base, origin xyz=-.025 0.043301270189222 .0 rpy=0 0 0
- joint f11_joint: parent f11_slot -> f11_base
- joint f12_joint: mimic joint=f11_joint multiplier=1 offset=-.25 -> joint=f11_joint multiplier=2 offset=-.25
- joint f21_joint: parent f21_slot -> f21_base
- joint f31_joint: parent f31_slot -> f31_base

File: assets/ur5/model.urdf (robot description, URDF)
Before this commit: robot universal_robot, 7 links, 6 joints
Links:
- added link ee_link; collision box size=0.01 0.01 0.01
Joints:
- added joint ee_fixed_joint: type fixed, parent wrist_3_link, child ee_link, origin xyz=0.0 0.0823 0.0 rpy=0.0 0.0 3.1415
- joint shoulder_lift_joint: limit lower=0 upper=3.14159 effort=150.0 velocity=3.15 -> lower=-2 upper=0 effort=150.0 velocity=3.15

Commit message: added limitation to movement space, next phase adding reward phase

File: assets/grippers/2f_1j.urdf (robot description, URDF)
Before this commit: robot gripper_2f_1j, 5 links, 4 joints
Links:
- added link f12_slot; visual sphere radius=.015
- added link f22_slot; visual sphere radius=.015
Joints:
- added joint f12_slot_joint: type fixed, parent f11, child f12_slot, origin xyz=0 0 .1 rpy=0 0 0
- added joint f22_slot_joint: type fixed, parent f21, child f22_slot, origin xyz=0 0 .1 rpy=0 0 0

File: assets/grippers/2f_2j.urdf (robot description, URDF)
Before this commit: robot gripper_2f_2j, 9 links, 8 joints
Links:
- added link f13_slot; visual sphere radius=.015
- added link f23_slot; visual sphere radius=.015
Joints:
- added joint f13_slot_joint: type fixed, parent f12, child f13_slot, origin xyz=0 0 .05 rpy=0 0 0
- added joint f23_slot_joint: type fixed, parent f22, child f23_slot, origin xyz=0 0 .05 rpy=0 0 0

File: assets/grippers/3f_1j.urdf (robot description, URDF)
Before this commit: robot gripper_3f_1j, 7 links, 6 joints
Links:
- added link f12_slot; visual sphere radius=.015
- added link f22_slot; visual sphere radius=.015
- added link f32_slot; visual sphere radius=.015
Joints:
- added joint f12_slot_joint: type fixed, parent f11, child f12_slot, origin xyz=0 0 .1 rpy=0 0 0
- added joint f22_slot_joint: type fixed, parent f21, child f22_slot, origin xyz=0 0 .1 rpy=0 0 0
- added joint f32_slot_joint: type fixed, parent f31, child f32_slot, origin xyz=0 0 .1 rpy=0 0 0

File: assets/ur5/model copy.urdf (robot description, URDF)
Before this commit: robot ur5_2f1j, 15 links, 14 joints
Links:
- removed link f11
- removed link f11_base
- removed link f12_slot
- removed link f21
- removed link f21_base
- removed link f22_slot
- removed link palm
- link ee_link: mass 0. -> None
Joints:
- removed joint f11_base_joint
- removed joint f11_joint
- removed joint f12_slot_joint
- removed joint f21_base_joint
- removed joint f21_joint
- removed joint f22_slot_joint
- removed joint palm_ee_joint
- joint ee_fixed_joint: origin xyz=0.0 0.0823. 0. rpy=0.0 0.0 1.57079632679 -> xyz=0.0 0.0823 0.0 rpy=0.0 0.0 3.1415
- joint elbow_joint: limit lower=-.5159265359 upper=2.14159265359 effort=150.0 velocity=3.15 -> lower=-3.14159265359 upper=3.14159265359 effort=150.0 velocity=3.15
- joint shoulder_pan_joint: limit lower=-.5 upper=.5 effort=150.0 velocity=3.15 -> lower=-6.28318530718 upper=6.28318530718 effort=150.0 velocity=3.15
- joint wrist_1_joint: limit lower=-3.28318530718 upper=6.28318530718 effort=28.0 velocity=3.2 -> lower=-6.28318530718 upper=6.28318530718 effort=28.0 velocity=3.2

File: assets/ur5_w_gripper/2f_2j.urdf (robot description, URDF)
Before this commit: robot ur5_2f1j, 17 links, 16 joints
Links:
- added link f13_slot; visual sphere radius=.015
- added link f23_slot; visual sphere radius=.015
Joints:
- added joint f13_slot_joint: type fixed, parent f12, child f13_slot, origin xyz=0 0 .05 rpy=0 0 0
- added joint f23_slot_joint: type fixed, parent f22, child f23_slot, origin xyz=0 0 .05 rpy=0 0 0

File: assets/ur5_w_gripper/3f_1j.urdf (robot description, URDF)
Before this commit: robot ur5_2f1j, 15 links, 14 joints
Links:
- added link f12; collision cylinder length=.05 radius=.01; visual cylinder length=.05 radius=.01
- added link f12_slot; visual sphere radius=.015
- added link f22; collision cylinder length=.05 radius=.01; visual cylinder length=.05 radius=.01
- added link f22_slot; visual sphere radius=.015
- added link f32; collision cylinder length=.05 radius=.01; visual cylinder length=.05 radius=.01
- added link f32_slot; visual sphere radius=.015
- link f11: geometry collision cylinder length=.05 radius=.01; visual cylinder length=.05 radius=.01
- link f21: geometry collision cylinder length=.05 radius=.01; visual cylinder length=.05 radius=.01
- link f31: geometry collision cylinder length=.05 radius=.01; visual cylinder length=.05 radius=.01
Joints:
- added joint f12_joint: type revolute, parent f12_slot, child f12, origin xyz=0 0 .0 rpy=0 -.0 0, axis 0 1 0, limit lower=-.65 upper=.0 effort=30 velocity=2.0, mimic joint=f11_joint multiplier=2 offset=-.25
- added joint f12_slot_joint: type fixed, parent f11, child f12_slot, origin xyz=0 0 .05 rpy=0 0 0
- added joint f22_joint: type revolute, parent f22_slot, child f22, origin xyz=0 0 .0 rpy=0 -.0 0, axis 1 -1 0, limit lower=-.65 upper=.0 effort=30 velocity=2.0, mimic joint=f21_joint multiplier=1 offset=-.25
- added joint f22_slot_joint: type fixed, parent f21, child f22_slot, origin xyz=0 0 .05 rpy=0 0 0
- added joint f32_joint: type revolute, parent f32_slot, child f32, origin xyz=0 0 .0 rpy=0 -.0 0, axis -1 -1 0, limit lower=-.65 upper=.0 effort=30 velocity=2.0, mimic joint=f31_joint multiplier=1 offset=-.25
- added joint f32_slot_joint: type fixed, parent f31, child f32_slot, origin xyz=0 0 .05 rpy=0 0 0
- joint f11_joint: limit lower=-.65 upper=.25 effort=30 velocity=2.0 -> lower=-.4 upper=.25 effort=30 velocity=2.0
- joint f21_joint: limit lower=-.65 upper=.25 effort=30 velocity=2.0 -> lower=-.4 upper=.25 effort=30 velocity=2.0; mimic joint=f11_joint multiplier=1 -> (none)
- joint f31_joint: limit lower=-.65 upper=.25 effort=30 velocity=2.0 -> lower=-.4 upper=.25 effort=30 velocity=2.0; mimic joint=f11_joint multiplier=1 -> (none)

File: assets/ur5_w_gripper/3f_2j.urdf (robot description, URDF)
Before this commit: robot ur5_2f1j, 21 links, 20 joints
Links:
- added link f13_slot; visual sphere radius=.015
- added link f23_slot; visual sphere radius=.015
- added link f33_slot; visual sphere radius=.015
Joints:
- added joint f13_slot_joint: type fixed, parent f12, child f13_slot, origin xyz=0 0 .05 rpy=0 0 0
- added joint f23_slot_joint: type fixed, parent f22, child f23_slot, origin xyz=0 0 .05 rpy=0 0 0
- added joint f33_slot_joint: type fixed, parent f32, child f33_slot, origin xyz=0 0 .05 rpy=0 0 0
- joint shoulder_lift_joint: limit lower=-2 upper=0 effort=150.0 velocity=3.15 -> lower=-3.14 upper=3.14 effort=150.0 velocity=3.15
