Commit message: changed reward definition, distance

File: assets/3f_2j.urdf (robot description, URDF)
Before this commit: robot ur5_3f2j, 24 links, 23 joints
Joints:
- joint shoulder_lift_joint: limit lower=-3.14 upper=3.14 effort=150.0 velocity=3.15 -> lower=-3.14159265359 upper=3.14159265359 effort=150.0 velocity=3.15
- joint shoulder_pan_joint: limit lower=-3.142 upper=3.142 effort=150.0 velocity=3.15 -> lower=-3.14159265359 upper=3.14159265359 effort=150.0 velocity=3.15

Commit message: update

File: assets/3f_2j.urdf (robot description, URDF)
Before this commit: robot ur5_3f2j, 24 links, 23 joints
Joints:
- joint f12_joint: limit lower=-0.65 upper=0.0 effort=30.0 velocity=2.0 -> lower=-0.4 upper=0.0 effort=30.0 velocity=2.0
- joint f22_joint: limit lower=-0.65 upper=0.0 effort=30.0 velocity=2.0 -> lower=-0.4 upper=0.0 effort=30.0 velocity=2.0
- joint f32_joint: limit lower=-0.65 upper=0. effort=30.0 velocity=2.0 -> lower=-0.4 upper=0. effort=30.0 velocity=2.0

File: assets/gen_gripper/3f_2j/robot_0/model.urdf (robot description, URDF)
Before this commit: robot gripper_3f_2j, 13 links, 12 joints
Links:
- added link base_link, mass 4.0; collision mesh filename=meshes/ur5/collision/base.stl; visual mesh filename=meshes/ur5/visual/base.obj
- added link ee_link, mass 0.0; collision box size=0.01 0.01 0.01
- added link f13_slot, mass 0.0; visual sphere radius=0.015
- added link f23_slot, mass 0.0; visual sphere radius=0.015
- added link f33_slot, mass 0.0; visual sphere radius=0.015
- added link forearm_link, mass 2.275; collision mesh filename=meshes/ur5/collision/forearm.stl; visual mesh filename=meshes/ur5/visual/forearm.obj
- added link shoulder_link, mass 3.7; collision mesh filename=meshes/ur5/collision/shoulder.stl; visual mesh filename=meshes/ur5/visual/shoulder.obj
- added link upper_arm_link, mass 8.393; collision mesh filename=meshes/ur5/collision/upperarm.stl; visual mesh filename=meshes/ur5/visual/upperarm.obj
- added link wrist_1_link, mass 1.219; collision mesh filename=meshes/ur5/collision/wrist1.stl; visual mesh filename=meshes/ur5/visual/wrist1.obj
- added link wrist_2_link, mass 1.219; collision mesh filename=meshes/ur5/collision/wrist2.stl; visual mesh filename=meshes/ur5/visual/wrist2.obj
- added link wrist_3_link, mass 0.1879; collision mesh filename=meshes/ur5/collision/wrist3.stl; visual mesh filename=meshes/ur5/visual/wrist3.obj
- link f11: geometry collision cylinder length=0.16725651908061906 radius=0.01920251154799855; visual cylinder length=0.16725651908061906 radius=0.01920251154799855
- link f11_base: mass 1.0 -> 0.01
- link f12: geometry collision cylinder length=0.1356882724355507 radius=0.01920251154799855; visual cylinder length=0.1356882724355507 radius=0.01920251154799855
- link f12_slot: mass 1.0 -> 0.01
- link f21: geometry collision cylinder length=0.16725651908061906 radius=0.01920251154799855; visual cylinder length=0.16725651908061906 radius=0.01920251154799855
- link f21_base: mass 1.0 -> 0.01
- link f22: geometry collision cylinder length=0.1356882724355507 radius=0.01920251154799855; visual cylinder length=0.1356882724355507 radius=0.01920251154799855
- link f22_slot: mass 1.0 -> 0.01
- link f31: geometry collision cylinder length=0.16725651908061906 radius=0.01920251154799855; visual cylinder length=0.16725651908061906 radius=0.01920251154799855
- link f31_base: mass 1.0 -> 0.0
- link f32: geometry collision cylinder length=0.1356882724355507 radius=0.01920251154799855; visual cylinder length=0.1356882724355507 radius=0.01920251154799855
- link f32_slot: mass 1.0 -> 0.0
Joints:
- added joint ee_fixed_joint: type fixed, parent wrist_3_link, child ee_link, origin xyz=0.0 0.0823 0.0 rpy=0.0 0.0 1.57079632679, axis 1. 0. 0.
- added joint elbow_joint: type revolute, parent upper_arm_link, child forearm_link, origin xyz=0.0 -0.1197 0.425 rpy=0.0 0.0 0.0, axis 0. 1. 0., limit lower=-3.14159265359 upper=3.14159265359 effort=150.0 velocity=3.15
- added joint f13_slot_joint: type fixed, parent f12, child f13_slot, origin xyz=0.0 0.0 0.05 rpy=0.0 0.0 0.0, axis 1. 0. 0.
- added joint f23_slot_joint: type fixed, parent f22, child f23_slot, origin xyz=0.0 0.0 0.05 rpy=0.0 0.0 0.0, axis 1. 0. 0.
- added joint f33_slot_joint: type fixed, parent f32, child f33_slot, origin xyz=0.0 0.0 0.05 rpy=0.0 0.0 0.0, axis 1. 0. 0.
- added joint palm_ee_joint: type fixed, parent ee_link, child palm, origin xyz=0.0 0.0 0.0 rpy=3.14 1.5699999999999876 3.14, axis 1. 0. 0.
- added joint shoulder_lift_joint: type revolute, parent shoulder_link, child upper_arm_link, origin xyz=0.0 0.13585 0.0 rpy=0.0 1.5707963267948966 0.0, axis 0. 1. 0., limit lower=-3.14159265359 upper=3.14159265359 effort=150.0 velocity=3.15
- added joint shoulder_pan_joint: type revolute, parent base_link, child shoulder_link, origin xyz=0.0 0.0 0.089159 rpy=0.0 0.0 0.0, axis 0. 0. 1., limit lower=-3.14159265359 upper=3.14159265359 effort=150.0 velocity=3.15
- added joint wrist_1_joint: type revolute, parent forearm_link, child wrist_1_link, origin xyz=0.0 0.0 0.39225 rpy=0.0 1.5707963267948966 0.0, axis 0. 1. 0., limit lower=-6.28318530718 upper=6.28318530718 effort=28.0 velocity=3.2
- added joint wrist_2_joint: type revolute, parent wrist_1_link, child wrist_2_link, origin xyz=0.0 0.093 0.0 rpy=0.0 0.0 0.0, axis 0. 0. 1., limit lower=-6.28318530718 upper=6.28318530718 effort=28.0 velocity=3.2
- added joint wrist_3_joint: type revolute, parent wrist_2_link, child wrist_3_link, origin xyz=0.0 0.0 0.09465 rpy=0.0 0.0 0.0, axis 0. 1. 0., limit lower=-6.28318530718 upper=6.28318530718 effort=28.0 velocity=3.2
- joint f12_joint: limit lower=-0.65 upper=0.0 effort=30.0 velocity=2.0 -> lower=-0.4 upper=0.0 effort=30.0 velocity=2.0
- joint f12_slot_joint: origin xyz=0.0 0.0 0.034655890843647445 rpy=0.0 0.0 0.0 -> xyz=0.0 0.0 0.16725651908061906 rpy=0.0 0.0 0.0
- joint f22_joint: limit lower=-0.65 upper=0.0 effort=30.0 velocity=2.0 -> lower=-0.4 upper=0.0 effort=30.0 velocity=2.0
- joint f22_slot_joint: origin xyz=0.0 0.0 0.034655890843647445 rpy=0.0 0.0 0.0 -> xyz=0.0 0.0 0.16725651908061906 rpy=0.0 0.0 0.0
- joint f32_joint: limit lower=-0.65 upper=0.0 effort=30.0 velocity=2.0 -> lower=-0.4 upper=0.0 effort=30.0 velocity=2.0; origin xyz=0.0 0.0 0.0 rpy=0.0 -0.0 0.0 -> xyz=0.0 0.0 0.0 rpy=0.0 0.0 0.0
- joint f32_slot_joint: origin xyz=0.0 0.0 0.034655890843647445 rpy=0.0 0.0 0.0 -> xyz=0.0 0.0 0.16725651908061906 rpy=0.0 0.0 0.0

File: assets/gen_gripper/3f_2j/robot_1/model.urdf (robot description, URDF)
Before this commit: robot gripper_3f_2j, 13 links, 12 joints
Links:
- added link base_link, mass 4.0; collision mesh filename=meshes/ur5/collision/base.stl; visual mesh filename=meshes/ur5/visual/base.obj
- added link ee_link, mass 0.0; collision box size=0.01 0.01 0.01
- added link f13_slot, mass 0.0; visual sphere radius=0.015
- added link f23_slot, mass 0.0; visual sphere radius=0.015
- added link f33_slot, mass 0.0; visual sphere radius=0.015
- added link forearm_link, mass 2.275; collision mesh filename=meshes/ur5/collision/forearm.stl; visual mesh filename=meshes/ur5/visual/forearm.obj
- added link shoulder_link, mass 3.7; collision mesh filename=meshes/ur5/collision/shoulder.stl; visual mesh filename=meshes/ur5/visual/shoulder.obj
- added link upper_arm_link, mass 8.393; collision mesh filename=meshes/ur5/collision/upperarm.stl; visual mesh filename=meshes/ur5/visual/upperarm.obj
- added link wrist_1_link, mass 1.219; collision mesh filename=meshes/ur5/collision/wrist1.stl; visual mesh filename=meshes/ur5/visual/wrist1.obj
- added link wrist_2_link, mass 1.219; collision mesh filename=meshes/ur5/collision/wrist2.stl; visual mesh filename=meshes/ur5/visual/wrist2.obj
- added link wrist_3_link, mass 0.1879; collision mesh filename=meshes/ur5/collision/wrist3.stl; visual mesh filename=meshes/ur5/visual/wrist3.obj
- link f11: geometry collision cylinder length=0.12832623444581243 radius=0.021730822336329614; visual cylinder length=0.12832623444581243 radius=0.021730822336329614
- link f11_base: mass 1.0 -> 0.01
- link f12: geometry collision cylinder length=0.15766021378464734 radius=0.021730822336329614; visual cylinder length=0.15766021378464734 radius=0.021730822336329614
- link f12_slot: mass 1.0 -> 0.01
- link f21: geometry collision cylinder length=0.12832623444581243 radius=0.021730822336329614; visual cylinder length=0.12832623444581243 radius=0.021730822336329614
- link f21_base: mass 1.0 -> 0.01
- link f22: geometry collision cylinder length=0.15766021378464734 radius=0.021730822336329614; visual cylinder length=0.15766021378464734 radius=0.021730822336329614
- link f22_slot: mass 1.0 -> 0.01
- link f31: geometry collision cylinder length=0.12832623444581243 radius=0.021730822336329614; visual cylinder length=0.12832623444581243 radius=0.021730822336329614
- link f31_base: mass 1.0 -> 0.0
- link f32: geometry collision cylinder length=0.15766021378464734 radius=0.021730822336329614; visual cylinder length=0.15766021378464734 radius=0.021730822336329614
- link f32_slot: mass 1.0 -> 0.0
Joints:
- added joint ee_fixed_joint: type fixed, parent wrist_3_link, child ee_link, origin xyz=0.0 0.0823 0.0 rpy=0.0 0.0 1.57079632679, axis 1. 0. 0.
- added joint elbow_joint: type revolute, parent upper_arm_link, child forearm_link, origin xyz=0.0 -0.1197 0.425 rpy=0.0 0.0 0.0, axis 0. 1. 0., limit lower=-3.14159265359 upper=3.14159265359 effort=150.0 velocity=3.15
- added joint f13_slot_joint: type fixed, parent f12, child f13_slot, origin xyz=0.0 0.0 0.05 rpy=0.0 0.0 0.0, axis 1. 0. 0.
- added joint f23_slot_joint: type fixed, parent f22, child f23_slot, origin xyz=0.0 0.0 0.05 rpy=0.0 0.0 0.0, axis 1. 0. 0.
- added joint f33_slot_joint: type fixed, parent f32, child f33_slot, origin xyz=0.0 0.0 0.05 rpy=0.0 0.0 0.0, axis 1. 0. 0.
- added joint palm_ee_joint: type fixed, parent ee_link, child palm, origin xyz=0.0 0.0 0.0 rpy=3.14 1.5699999999999876 3.14, axis 1. 0. 0.
- added joint shoulder_lift_joint: type revolute, parent shoulder_link, child upper_arm_link, origin xyz=0.0 0.13585 0.0 rpy=0.0 1.5707963267948966 0.0, axis 0. 1. 0., limit lower=-3.14159265359 upper=3.14159265359 effort=150.0 velocity=3.15
- added joint shoulder_pan_joint: type revolute, parent base_link, child shoulder_link, origin xyz=0.0 0.0 0.089159 rpy=0.0 0.0 0.0, axis 0. 0. 1., limit lower=-3.14159265359 upper=3.14159265359 effort=150.0 velocity=3.15
- added joint wrist_1_joint: type revolute, parent forearm_link, child wrist_1_link, origin xyz=0.0 0.0 0.39225 rpy=0.0 1.5707963267948966 0.0, axis 0. 1. 0., limit lower=-6.28318530718 upper=6.28318530718 effort=28.0 velocity=3.2
- added joint wrist_2_joint: type revolute, parent wrist_1_link, child wrist_2_link, origin xyz=0.0 0.093 0.0 rpy=0.0 0.0 0.0, axis 0. 0. 1., limit lower=-6.28318530718 upper=6.28318530718 effort=28.0 velocity=3.2
- added joint wrist_3_joint: type revolute, parent wrist_2_link, child wrist_3_link, origin xyz=0.0 0.0 0.09465 rpy=0.0 0.0 0.0, axis 0. 1. 0., limit lower=-6.28318530718 upper=6.28318530718 effort=28.0 velocity=3.2
- joint f12_joint: limit lower=-0.65 upper=0.0 effort=30.0 velocity=2.0 -> lower=-0.4 upper=0.0 effort=30.0 velocity=2.0
- joint f12_slot_joint: origin xyz=0.0 0.0 0.18208313279565405 rpy=0.0 0.0 0.0 -> xyz=0.0 0.0 0.12832623444581243 rpy=0.0 0.0 0.0
- joint f22_joint: limit lower=-0.65 upper=0.0 effort=30.0 velocity=2.0 -> lower=-0.4 upper=0.0 effort=30.0 velocity=2.0
- joint f22_slot_joint: origin xyz=0.0 0.0 0.18208313279565405 rpy=0.0 0.0 0.0 -> xyz=0.0 0.0 0.12832623444581243 rpy=0.0 0.0 0.0
- joint f32_joint: limit lower=-0.65 upper=0.0 effort=30.0 velocity=2.0 -> lower=-0.4 upper=0.0 effort=30.0 velocity=2.0; origin xyz=0.0 0.0 0.0 rpy=0.0 -0.0 0.0 -> xyz=0.0 0.0 0.0 rpy=0.0 0.0 0.0
- joint f32_slot_joint: origin xyz=0.0 0.0 0.18208313279565405 rpy=0.0 0.0 0.0 -> xyz=0.0 0.0 0.12832623444581243 rpy=0.0 0.0 0.0

File: assets/gen_gripper/3f_2j/robot_2/model.urdf (robot description, URDF)
Before this commit: robot gripper_3f_2j, 13 links, 12 joints
Links:
- added link base_link, mass 4.0; collision mesh filename=meshes/ur5/collision/base.stl; visual mesh filename=meshes/ur5/visual/base.obj
- added link ee_link, mass 0.0; collision box size=0.01 0.01 0.01
- added link f13_slot, mass 0.0; visual sphere radius=0.015
- added link f23_slot, mass 0.0; visual sphere radius=0.015
- added link f33_slot, mass 0.0; visual sphere radius=0.015
- added link forearm_link, mass 2.275; collision mesh filename=meshes/ur5/collision/forearm.stl; visual mesh filename=meshes/ur5/visual/forearm.obj
- added link shoulder_link, mass 3.7; collision mesh filename=meshes/ur5/collision/shoulder.stl; visual mesh filename=meshes/ur5/visual/shoulder.obj
- added link upper_arm_link, mass 8.393; collision mesh filename=meshes/ur5/collision/upperarm.stl; visual mesh filename=meshes/ur5/visual/upperarm.obj
- added link wrist_1_link, mass 1.219; collision mesh filename=meshes/ur5/collision/wrist1.stl; visual mesh filename=meshes/ur5/visual/wrist1.obj
- added link wrist_2_link, mass 1.219; collision mesh filename=meshes/ur5/collision/wrist2.stl; visual mesh filename=meshes/ur5/visual/wrist2.obj
- added link wrist_3_link, mass 0.1879; collision mesh filename=meshes/ur5/collision/wrist3.stl; visual mesh filename=meshes/ur5/visual/wrist3.obj
- link f11: geometry collision cylinder length=0.03001944371894863 radius=0.02041945892504144; visual cylinder length=0.03001944371894863 radius=0.02041945892504144
- link f11_base: mass 1.0 -> 0.01
- link f12: geometry collision cylinder length=0.05887117132597672 radius=0.02041945892504144; visual cylinder length=0.05887117132597672 radius=0.02041945892504144
- link f12_slot: mass 1.0 -> 0.01
- link f21: geometry collision cylinder length=0.03001944371894863 radius=0.02041945892504144; visual cylinder length=0.03001944371894863 radius=0.02041945892504144
- link f21_base: mass 1.0 -> 0.01
- link f22: geometry collision cylinder length=0.05887117132597672 radius=0.02041945892504144; visual cylinder length=0.05887117132597672 radius=0.02041945892504144
- link f22_slot: mass 1.0 -> 0.01
- link f31: geometry collision cylinder length=0.03001944371894863 radius=0.02041945892504144; visual cylinder length=0.03001944371894863 radius=0.02041945892504144
- link f31_base: mass 1.0 -> 0.0
- link f32: geometry collision cylinder length=0.05887117132597672 radius=0.02041945892504144; visual cylinder length=0.05887117132597672 radius=0.02041945892504144
- link f32_slot: mass 1.0 -> 0.0
Joints:
- added joint ee_fixed_joint: type fixed, parent wrist_3_link, child ee_link, origin xyz=0.0 0.0823 0.0 rpy=0.0 0.0 1.57079632679, axis 1. 0. 0.
- added joint elbow_joint: type revolute, parent upper_arm_link, child forearm_link, origin xyz=0.0 -0.1197 0.425 rpy=0.0 0.0 0.0, axis 0. 1. 0., limit lower=-3.14159265359 upper=3.14159265359 effort=150.0 velocity=3.15
- added joint f13_slot_joint: type fixed, parent f12, child f13_slot, origin xyz=0.0 0.0 0.05 rpy=0.0 0.0 0.0, axis 1. 0. 0.
- added joint f23_slot_joint: type fixed, parent f22, child f23_slot, origin xyz=0.0 0.0 0.05 rpy=0.0 0.0 0.0, axis 1. 0. 0.
- added joint f33_slot_joint: type fixed, parent f32, child f33_slot, origin xyz=0.0 0.0 0.05 rpy=0.0 0.0 0.0, axis 1. 0. 0.
- added joint palm_ee_joint: type fixed, parent ee_link, child palm, origin xyz=0.0 0.0 0.0 rpy=3.14 1.5699999999999876 3.14, axis 1. 0. 0.
- added joint shoulder_lift_joint: type revolute, parent shoulder_link, child upper_arm_link, origin xyz=0.0 0.13585 0.0 rpy=0.0 1.5707963267948966 0.0, axis 0. 1. 0., limit lower=-3.14159265359 upper=3.14159265359 effort=150.0 velocity=3.15
- added joint shoulder_pan_joint: type revolute, parent base_link, child shoulder_link, origin xyz=0.0 0.0 0.089159 rpy=0.0 0.0 0.0, axis 0. 0. 1., limit lower=-3.14159265359 upper=3.14159265359 effort=150.0 velocity=3.15
- added joint wrist_1_joint: type revolute, parent forearm_link, child wrist_1_link, origin xyz=0.0 0.0 0.39225 rpy=0.0 1.5707963267948966 0.0, axis 0. 1. 0., limit lower=-6.28318530718 upper=6.28318530718 effort=28.0 velocity=3.2
- added joint wrist_2_joint: type revolute, parent wrist_1_link, child wrist_2_link, origin xyz=0.0 0.093 0.0 rpy=0.0 0.0 0.0, axis 0. 0. 1., limit lower=-6.28318530718 upper=6.28318530718 effort=28.0 velocity=3.2
- added joint wrist_3_joint: type revolute, parent wrist_2_link, child wrist_3_link, origin xyz=0.0 0.0 0.09465 rpy=0.0 0.0 0.0, axis 0. 1. 0., limit lower=-6.28318530718 upper=6.28318530718 effort=28.0 velocity=3.2
- joint f12_joint: limit lower=-0.65 upper=0.0 effort=30.0 velocity=2.0 -> lower=-0.4 upper=0.0 effort=30.0 velocity=2.0
- joint f12_slot_joint: origin xyz=0.0 0.0 0.1301819412735583 rpy=0.0 0.0 0.0 -> xyz=0.0 0.0 0.03001944371894863 rpy=0.0 0.0 0.0
- joint f22_joint: limit lower=-0.65 upper=0.0 effort=30.0 velocity=2.0 -> lower=-0.4 upper=0.0 effort=30.0 velocity=2.0
- joint f22_slot_joint: origin xyz=0.0 0.0 0.1301819412735583 rpy=0.0 0.0 0.0 -> xyz=0.0 0.0 0.03001944371894863 rpy=0.0 0.0 0.0
- joint f32_joint: limit lower=-0.65 upper=0.0 effort=30.0 velocity=2.0 -> lower=-0.4 upper=0.0 effort=30.0 velocity=2.0; origin xyz=0.0 0.0 0.0 rpy=0.0 -0.0 0.0 -> xyz=0.0 0.0 0.0 rpy=0.0 0.0 0.0
- joint f32_slot_joint: origin xyz=0.0 0.0 0.1301819412735583 rpy=0.0 0.0 0.0 -> xyz=0.0 0.0 0.03001944371894863 rpy=0.0 0.0 0.0

File: assets/gen_gripper/3f_2j/robot_3/model.urdf (robot description, URDF)
Before this commit: robot gripper_3f_2j, 13 links, 12 joints
Links:
- added link base_link, mass 4.0; collision mesh filename=meshes/ur5/collision/base.stl; visual mesh filename=meshes/ur5/visual/base.obj
- added link ee_link, mass 0.0; collision box size=0.01 0.01 0.01
- added link f13_slot, mass 0.0; visual sphere radius=0.015
- added link f23_slot, mass 0.0; visual sphere radius=0.015
- added link f33_slot, mass 0.0; visual sphere radius=0.015
- added link forearm_link, mass 2.275; collision mesh filename=meshes/ur5/collision/forearm.stl; visual mesh filename=meshes/ur5/visual/forearm.obj
- added link shoulder_link, mass 3.7; collision mesh filename=meshes/ur5/collision/shoulder.stl; visual mesh filename=meshes/ur5/visual/shoulder.obj
- added link upper_arm_link, mass 8.393; collision mesh filename=meshes/ur5/collision/upperarm.stl; visual mesh filename=meshes/ur5/visual/upperarm.obj
- added link wrist_1_link, mass 1.219; collision mesh filename=meshes/ur5/collision/wrist1.stl; visual mesh filename=meshes/ur5/visual/wrist1.obj
- added link wrist_2_link, mass 1.219; collision mesh filename=meshes/ur5/collision/wrist2.stl; visual mesh filename=meshes/ur5/visual/wrist2.obj
- added link wrist_3_link, mass 0.1879; collision mesh filename=meshes/ur5/collision/wrist3.stl; visual mesh filename=meshes/ur5/visual/wrist3.obj
- link f11: geometry collision cylinder length=0.06597677972001004 radius=0.0276953963125881; visual cylinder length=0.06597677972001004 radius=0.0276953963125881
- link f11_base: mass 1.0 -> 0.01
- link f12: geometry collision cylinder length=0.0332923828379505 radius=0.0276953963125881; visual cylinder length=0.0332923828379505 radius=0.0276953963125881
- link f12_slot: mass 1.0 -> 0.01
- link f21: geometry collision cylinder length=0.06597677972001004 radius=0.0276953963125881; visual cylinder length=0.06597677972001004 radius=0.0276953963125881
- link f21_base: mass 1.0 -> 0.01
- link f22: geometry collision cylinder length=0.0332923828379505 radius=0.0276953963125881; visual cylinder length=0.0332923828379505 radius=0.0276953963125881
- link f22_slot: mass 1.0 -> 0.01
- link f31: geometry collision cylinder length=0.06597677972001004 radius=0.0276953963125881; visual cylinder length=0.06597677972001004 radius=0.0276953963125881
- link f31_base: mass 1.0 -> 0.0
- link f32: geometry collision cylinder length=0.0332923828379505 radius=0.0276953963125881; visual cylinder length=0.0332923828379505 radius=0.0276953963125881
- link f32_slot: mass 1.0 -> 0.0
Joints:
- added joint ee_fixed_joint: type fixed, parent wrist_3_link, child ee_link, origin xyz=0.0 0.0823 0.0 rpy=0.0 0.0 1.57079632679, axis 1. 0. 0.
- added joint elbow_joint: type revolute, parent upper_arm_link, child forearm_link, origin xyz=0.0 -0.1197 0.425 rpy=0.0 0.0 0.0, axis 0. 1. 0., limit lower=-3.14159265359 upper=3.14159265359 effort=150.0 velocity=3.15
- added joint f13_slot_joint: type fixed, parent f12, child f13_slot, origin xyz=0.0 0.0 0.05 rpy=0.0 0.0 0.0, axis 1. 0. 0.
- added joint f23_slot_joint: type fixed, parent f22, child f23_slot, origin xyz=0.0 0.0 0.05 rpy=0.0 0.0 0.0, axis 1. 0. 0.
- added joint f33_slot_joint: type fixed, parent f32, child f33_slot, origin xyz=0.0 0.0 0.05 rpy=0.0 0.0 0.0, axis 1. 0. 0.
- added joint palm_ee_joint: type fixed, parent ee_link, child palm, origin xyz=0.0 0.0 0.0 rpy=3.14 1.5699999999999876 3.14, axis 1. 0. 0.
- added joint shoulder_lift_joint: type revolute, parent shoulder_link, child upper_arm_link, origin xyz=0.0 0.13585 0.0 rpy=0.0 1.5707963267948966 0.0, axis 0. 1. 0., limit lower=-3.14159265359 upper=3.14159265359 effort=150.0 velocity=3.15
- added joint shoulder_pan_joint: type revolute, parent base_link, child shoulder_link, origin xyz=0.0 0.0 0.089159 rpy=0.0 0.0 0.0, axis 0. 0. 1., limit lower=-3.14159265359 upper=3.14159265359 effort=150.0 velocity=3.15
- added joint wrist_1_joint: type revolute, parent forearm_link, child wrist_1_link, origin xyz=0.0 0.0 0.39225 rpy=0.0 1.5707963267948966 0.0, axis 0. 1. 0., limit lower=-6.28318530718 upper=6.28318530718 effort=28.0 velocity=3.2
- added joint wrist_2_joint: type revolute, parent wrist_1_link, child wrist_2_link, origin xyz=0.0 0.093 0.0 rpy=0.0 0.0 0.0, axis 0. 0. 1., limit lower=-6.28318530718 upper=6.28318530718 effort=28.0 velocity=3.2
- added joint wrist_3_joint: type revolute, parent wrist_2_link, child wrist_3_link, origin xyz=0.0 0.0 0.09465 rpy=0.0 0.0 0.0, axis 0. 1. 0., limit lower=-6.28318530718 upper=6.28318530718 effort=28.0 velocity=3.2
- joint f12_joint: limit lower=-0.65 upper=0.0 effort=30.0 velocity=2.0 -> lower=-0.4 upper=0.0 effort=30.0 velocity=2.0
- joint f12_slot_joint: origin xyz=0.0 0.0 0.047548421118199145 rpy=0.0 0.0 0.0 -> xyz=0.0 0.0 0.06597677972001004 rpy=0.0 0.0 0.0
- joint f22_joint: limit lower=-0.65 upper=0.0 effort=30.0 velocity=2.0 -> lower=-0.4 upper=0.0 effort=30.0 velocity=2.0
- joint f22_slot_joint: origin xyz=0.0 0.0 0.047548421118199145 rpy=0.0 0.0 0.0 -> xyz=0.0 0.0 0.06597677972001004 rpy=0.0 0.0 0.0
- joint f32_joint: limit lower=-0.65 upper=0.0 effort=30.0 velocity=2.0 -> lower=-0.4 upper=0.0 effort=30.0 velocity=2.0; origin xyz=0.0 0.0 0.0 rpy=0.0 -0.0 0.0 -> xyz=0.0 0.0 0.0 rpy=0.0 0.0 0.0
- joint f32_slot_joint: origin xyz=0.0 0.0 0.047548421118199145 rpy=0.0 0.0 0.0 -> xyz=0.0 0.0 0.06597677972001004 rpy=0.0 0.0 0.0
