Commit message: env with diff arm

File: assets/gen_gripper/3f_2j/robot_0/model.urdf (robot description, URDF)
Before this commit: robot ur5_3f2j, 24 links, 23 joints
Links:
- link f11: geometry collision cylinder length=0.08651739020966667 radius=0.01068100461919942; visual cylinder length=0.08651739020966667 radius=0.01068100461919942
- link f12: geometry collision cylinder length=0.07351870041463854 radius=0.01068100461919942; visual cylinder length=0.07351870041463854 radius=0.01068100461919942
- link f21: geometry collision cylinder length=0.08651739020966667 radius=0.01068100461919942; visual cylinder length=0.08651739020966667 radius=0.01068100461919942
- link f22: geometry collision cylinder length=0.07351870041463854 radius=0.01068100461919942; visual cylinder length=0.07351870041463854 radius=0.01068100461919942
- link f31: geometry collision cylinder length=0.08651739020966667 radius=0.01068100461919942; visual cylinder length=0.08651739020966667 radius=0.01068100461919942
- link f32: geometry collision cylinder length=0.07351870041463854 radius=0.01068100461919942; visual cylinder length=0.07351870041463854 radius=0.01068100461919942
Joints:
- joint f12_slot_joint: origin xyz=0.0 0.0 0.16725651908061906 rpy=0.0 0.0 0.0 -> xyz=0.0 0.0 0.08651739020966667 rpy=0.0 0.0 0.0
- joint f13_slot_joint: origin xyz=0.0 0.0 0.05 rpy=0.0 0.0 0.0 -> xyz=0.0 0.0 0.07351870041463854 rpy=0.0 0.0 0.0
- joint f22_slot_joint: origin xyz=0.0 0.0 0.16725651908061906 rpy=0.0 0.0 0.0 -> xyz=0.0 0.0 0.08651739020966667 rpy=0.0 0.0 0.0
- joint f23_slot_joint: origin xyz=0.0 0.0 0.05 rpy=0.0 0.0 0.0 -> xyz=0.0 0.0 0.07351870041463854 rpy=0.0 0.0 0.0
- joint f32_slot_joint: origin xyz=0.0 0.0 0.16725651908061906 rpy=0.0 0.0 0.0 -> xyz=0.0 0.0 0.08651739020966667 rpy=0.0 0.0 0.0
- joint f33_slot_joint: origin xyz=0.0 0.0 0.05 rpy=0.0 0.0 0.0 -> xyz=0.0 0.0 0.07351870041463854 rpy=0.0 0.0 0.0

File: assets/gen_gripper/3f_2j/robot_1/model.urdf (robot description, URDF)
Before this commit: robot ur5_3f2j, 24 links, 23 joints
Links:
- link f11: geometry collision cylinder length=0.07048727300709923 radius=0.011692328934531846; visual cylinder length=0.07048727300709923 radius=0.011692328934531846
- link f12: geometry collision cylinder length=0.0825659703819136 radius=0.011692328934531846; visual cylinder length=0.0825659703819136 radius=0.011692328934531846
- link f21: geometry collision cylinder length=0.07048727300709923 radius=0.011692328934531846; visual cylinder length=0.07048727300709923 radius=0.011692328934531846
- link f22: geometry collision cylinder length=0.0825659703819136 radius=0.011692328934531846; visual cylinder length=0.0825659703819136 radius=0.011692328934531846
- link f31: geometry collision cylinder length=0.07048727300709923 radius=0.011692328934531846; visual cylinder length=0.07048727300709923 radius=0.011692328934531846
- link f32: geometry collision cylinder length=0.0825659703819136 radius=0.011692328934531846; visual cylinder length=0.0825659703819136 radius=0.011692328934531846
Joints:
- joint f12_slot_joint: origin xyz=0.0 0.0 0.12832623444581243 rpy=0.0 0.0 0.0 -> xyz=0.0 0.0 0.07048727300709923 rpy=0.0 0.0 0.0
- joint f13_slot_joint: origin xyz=0.0 0.0 0.05 rpy=0.0 0.0 0.0 -> xyz=0.0 0.0 0.0825659703819136 rpy=0.0 0.0 0.0
- joint f22_slot_joint: origin xyz=0.0 0.0 0.12832623444581243 rpy=0.0 0.0 0.0 -> xyz=0.0 0.0 0.07048727300709923 rpy=0.0 0.0 0.0
- joint f23_slot_joint: origin xyz=0.0 0.0 0.05 rpy=0.0 0.0 0.0 -> xyz=0.0 0.0 0.0825659703819136 rpy=0.0 0.0 0.0
- joint f32_slot_joint: origin xyz=0.0 0.0 0.12832623444581243 rpy=0.0 0.0 0.0 -> xyz=0.0 0.0 0.07048727300709923 rpy=0.0 0.0 0.0
- joint f33_slot_joint: origin xyz=0.0 0.0 0.05 rpy=0.0 0.0 0.0 -> xyz=0.0 0.0 0.0825659703819136 rpy=0.0 0.0 0.0

File: assets/gen_gripper/3f_2j/robot_2/model.urdf (robot description, URDF)
Before this commit: robot ur5_3f2j, 24 links, 23 joints
Links:
- link f11: geometry collision cylinder length=0.03000800623721414 radius=0.011167783570016576; visual cylinder length=0.03000800623721414 radius=0.011167783570016576
- link f12: geometry collision cylinder length=0.04188812936951982 radius=0.011167783570016576; visual cylinder length=0.04188812936951982 radius=0.011167783570016576
- link f21: geometry collision cylinder length=0.03000800623721414 radius=0.011167783570016576; visual cylinder length=0.03000800623721414 radius=0.011167783570016576
- link f22: geometry collision cylinder length=0.04188812936951982 radius=0.011167783570016576; visual cylinder length=0.04188812936951982 radius=0.011167783570016576
- link f31: geometry collision cylinder length=0.03000800623721414 radius=0.011167783570016576; visual cylinder length=0.03000800623721414 radius=0.011167783570016576
- link f32: geometry collision cylinder length=0.04188812936951982 radius=0.011167783570016576; visual cylinder length=0.04188812936951982 radius=0.011167783570016576
Joints:
- joint f12_slot_joint: origin xyz=0.0 0.0 0.03001944371894863 rpy=0.0 0.0 0.0 -> xyz=0.0 0.0 0.03000800623721414 rpy=0.0 0.0 0.0
- joint f13_slot_joint: origin xyz=0.0 0.0 0.05 rpy=0.0 0.0 0.0 -> xyz=0.0 0.0 0.04188812936951982 rpy=0.0 0.0 0.0
- joint f22_slot_joint: origin xyz=0.0 0.0 0.03001944371894863 rpy=0.0 0.0 0.0 -> xyz=0.0 0.0 0.03000800623721414 rpy=0.0 0.0 0.0
- joint f23_slot_joint: origin xyz=0.0 0.0 0.05 rpy=0.0 0.0 0.0 -> xyz=0.0 0.0 0.04188812936951982 rpy=0.0 0.0 0.0
- joint f32_slot_joint: origin xyz=0.0 0.0 0.03001944371894863 rpy=0.0 0.0 0.0 -> xyz=0.0 0.0 0.03000800623721414 rpy=0.0 0.0 0.0
- joint f33_slot_joint: origin xyz=0.0 0.0 0.05 rpy=0.0 0.0 0.0 -> xyz=0.0 0.0 0.04188812936951982 rpy=0.0 0.0 0.0

File: assets/gen_gripper/3f_2j/robot_3/model.urdf (robot description, URDF)
Before this commit: robot ur5_3f2j, 24 links, 23 joints
Links:
- link f11: geometry collision cylinder length=0.044813968120004134 radius=0.014078158525035238; visual cylinder length=0.044813968120004134 radius=0.014078158525035238
- link f12: geometry collision cylinder length=0.031355687050920796 radius=0.014078158525035238; visual cylinder length=0.031355687050920796 radius=0.014078158525035238
- link f21: geometry collision cylinder length=0.044813968120004134 radius=0.014078158525035238; visual cylinder length=0.044813968120004134 radius=0.014078158525035238
- link f22: geometry collision cylinder length=0.031355687050920796 radius=0.014078158525035238; visual cylinder length=0.031355687050920796 radius=0.014078158525035238
- link f31: geometry collision cylinder length=0.044813968120004134 radius=0.014078158525035238; visual cylinder length=0.044813968120004134 radius=0.014078158525035238
- link f32: geometry collision cylinder length=0.031355687050920796 radius=0.014078158525035238; visual cylinder length=0.031355687050920796 radius=0.014078158525035238
Joints:
- joint f12_slot_joint: origin xyz=0.0 0.0 0.06597677972001004 rpy=0.0 0.0 0.0 -> xyz=0.0 0.0 0.044813968120004134 rpy=0.0 0.0 0.0
- joint f13_slot_joint: origin xyz=0.0 0.0 0.05 rpy=0.0 0.0 0.0 -> xyz=0.0 0.0 0.031355687050920796 rpy=0.0 0.0 0.0
- joint f22_slot_joint: origin xyz=0.0 0.0 0.06597677972001004 rpy=0.0 0.0 0.0 -> xyz=0.0 0.0 0.044813968120004134 rpy=0.0 0.0 0.0
- joint f23_slot_joint: origin xyz=0.0 0.0 0.05 rpy=0.0 0.0 0.0 -> xyz=0.0 0.0 0.031355687050920796 rpy=0.0 0.0 0.0
- joint f32_slot_joint: origin xyz=0.0 0.0 0.06597677972001004 rpy=0.0 0.0 0.0 -> xyz=0.0 0.0 0.044813968120004134 rpy=0.0 0.0 0.0
- joint f33_slot_joint: origin xyz=0.0 0.0 0.05 rpy=0.0 0.0 0.0 -> xyz=0.0 0.0 0.031355687050920796 rpy=0.0 0.0 0.0

Commit message: updated with new range

File: assets/gen_gripper/3f_2j/robot_0/model.urdf (robot description, URDF)
Before this commit: robot ur5_3f2j, 24 links, 23 joints
Links:
- link f11: geometry collision cylinder length=0.075 radius=0.01068100461919942; visual cylinder length=0.075 radius=0.01068100461919942
- link f12: geometry collision cylinder length=0.075 radius=0.01068100461919942; visual cylinder length=0.075 radius=0.01068100461919942
- link f21: geometry collision cylinder length=0.075 radius=0.01068100461919942; visual cylinder length=0.075 radius=0.01068100461919942
- link f22: geometry collision cylinder length=0.075 radius=0.01068100461919942; visual cylinder length=0.075 radius=0.01068100461919942
- link f31: geometry collision cylinder length=0.075 radius=0.01068100461919942; visual cylinder length=0.075 radius=0.01068100461919942
- link f32: geometry collision cylinder length=0.075 radius=0.01068100461919942; visual cylinder length=0.075 radius=0.01068100461919942
Joints:
- joint f12_slot_joint: origin xyz=0.0 0.0 0.08651739020966667 rpy=0.0 0.0 0.0 -> xyz=0.0 0.0 0.075 rpy=0.0 0.0 0.0
- joint f13_slot_joint: origin xyz=0.0 0.0 0.07351870041463854 rpy=0.0 0.0 0.0 -> xyz=0.0 0.0 0.075 rpy=0.0 0.0 0.0
- joint f22_slot_joint: origin xyz=0.0 0.0 0.08651739020966667 rpy=0.0 0.0 0.0 -> xyz=0.0 0.0 0.075 rpy=0.0 0.0 0.0
- joint f23_slot_joint: origin xyz=0.0 0.0 0.07351870041463854 rpy=0.0 0.0 0.0 -> xyz=0.0 0.0 0.075 rpy=0.0 0.0 0.0
- joint f32_slot_joint: origin xyz=0.0 0.0 0.08651739020966667 rpy=0.0 0.0 0.0 -> xyz=0.0 0.0 0.075 rpy=0.0 0.0 0.0
- joint f33_slot_joint: origin xyz=0.0 0.0 0.07351870041463854 rpy=0.0 0.0 0.0 -> xyz=0.0 0.0 0.075 rpy=0.0 0.0 0.0

Commit message: updated with new env

File: assets/gen_gripper/3f_2j/robot_0/model.urdf (robot description, URDF)
Before this commit: robot ur5_3f2j, 24 links, 23 joints
Links:
- link f11: geometry collision cylinder length=0.06633260799192857 radius=0.01068100461919942; visual cylinder length=0.06633260799192857 radius=0.01068100461919942
- link f12: geometry collision cylinder length=0.05797630740941048 radius=0.01068100461919942; visual cylinder length=0.05797630740941048 radius=0.01068100461919942
- link f21: geometry collision cylinder length=0.06633260799192857 radius=0.01068100461919942; visual cylinder length=0.06633260799192857 radius=0.01068100461919942
- link f22: geometry collision cylinder length=0.05797630740941048 radius=0.01068100461919942; visual cylinder length=0.05797630740941048 radius=0.01068100461919942
- link f31: geometry collision cylinder length=0.06633260799192857 radius=0.01068100461919942; visual cylinder length=0.06633260799192857 radius=0.01068100461919942
- link f32: geometry collision cylinder length=0.05797630740941048 radius=0.01068100461919942; visual cylinder length=0.05797630740941048 radius=0.01068100461919942
Joints:
- joint f12_slot_joint: origin xyz=0.0 0.0 0.075 rpy=0.0 0.0 0.0 -> xyz=0.0 0.0 0.06633260799192857 rpy=0.0 0.0 0.0
- joint f13_slot_joint: origin xyz=0.0 0.0 0.075 rpy=0.0 0.0 0.0 -> xyz=0.0 0.0 0.05797630740941048 rpy=0.0 0.0 0.0
- joint f22_slot_joint: origin xyz=0.0 0.0 0.075 rpy=0.0 0.0 0.0 -> xyz=0.0 0.0 0.06633260799192857 rpy=0.0 0.0 0.0
- joint f23_slot_joint: origin xyz=0.0 0.0 0.075 rpy=0.0 0.0 0.0 -> xyz=0.0 0.0 0.05797630740941048 rpy=0.0 0.0 0.0
- joint f32_slot_joint: origin xyz=0.0 0.0 0.075 rpy=0.0 0.0 0.0 -> xyz=0.0 0.0 0.06633260799192857 rpy=0.0 0.0 0.0
- joint f33_slot_joint: origin xyz=0.0 0.0 0.075 rpy=0.0 0.0 0.0 -> xyz=0.0 0.0 0.05797630740941048 rpy=0.0 0.0 0.0

File: assets/gen_gripper/3f_2j/robot_1/model.urdf (robot description, URDF)
Before this commit: robot ur5_3f2j, 24 links, 23 joints
Links:
- link f11: geometry collision cylinder length=0.05602753264742093 radius=0.011692328934531846; visual cylinder length=0.05602753264742093 radius=0.011692328934531846
- link f12: geometry collision cylinder length=0.06379240953123017 radius=0.011692328934531846; visual cylinder length=0.06379240953123017 radius=0.011692328934531846
- link f21: geometry collision cylinder length=0.05602753264742093 radius=0.011692328934531846; visual cylinder length=0.05602753264742093 radius=0.011692328934531846
- link f22: geometry collision cylinder length=0.06379240953123017 radius=0.011692328934531846; visual cylinder length=0.06379240953123017 radius=0.011692328934531846
- link f31: geometry collision cylinder length=0.05602753264742093 radius=0.011692328934531846; visual cylinder length=0.05602753264742093 radius=0.011692328934531846
- link f32: geometry collision cylinder length=0.06379240953123017 radius=0.011692328934531846; visual cylinder length=0.06379240953123017 radius=0.011692328934531846
Joints:
- joint f12_slot_joint: origin xyz=0.0 0.0 0.07048727300709923 rpy=0.0 0.0 0.0 -> xyz=0.0 0.0 0.05602753264742093 rpy=0.0 0.0 0.0
- joint f13_slot_joint: origin xyz=0.0 0.0 0.0825659703819136 rpy=0.0 0.0 0.0 -> xyz=0.0 0.0 0.06379240953123017 rpy=0.0 0.0 0.0
- joint f22_slot_joint: origin xyz=0.0 0.0 0.07048727300709923 rpy=0.0 0.0 0.0 -> xyz=0.0 0.0 0.05602753264742093 rpy=0.0 0.0 0.0
- joint f23_slot_joint: origin xyz=0.0 0.0 0.0825659703819136 rpy=0.0 0.0 0.0 -> xyz=0.0 0.0 0.06379240953123017 rpy=0.0 0.0 0.0
- joint f32_slot_joint: origin xyz=0.0 0.0 0.07048727300709923 rpy=0.0 0.0 0.0 -> xyz=0.0 0.0 0.05602753264742093 rpy=0.0 0.0 0.0
- joint f33_slot_joint: origin xyz=0.0 0.0 0.0825659703819136 rpy=0.0 0.0 0.0 -> xyz=0.0 0.0 0.06379240953123017 rpy=0.0 0.0 0.0

File: assets/gen_gripper/3f_2j/robot_2/model.urdf (robot description, URDF)
Before this commit: robot ur5_3f2j, 24 links, 23 joints
Links:
- link f11: geometry collision cylinder length=0.03000514686678052 radius=0.011167783570016576; visual cylinder length=0.03000514686678052 radius=0.011167783570016576
- link f12: geometry collision cylinder length=0.0376423688804056 radius=0.011167783570016576; visual cylinder length=0.0376423688804056 radius=0.011167783570016576
- link f21: geometry collision cylinder length=0.03000514686678052 radius=0.011167783570016576; visual cylinder length=0.03000514686678052 radius=0.011167783570016576
- link f22: geometry collision cylinder length=0.0376423688804056 radius=0.011167783570016576; visual cylinder length=0.0376423688804056 radius=0.011167783570016576
- link f31: geometry collision cylinder length=0.03000514686678052 radius=0.011167783570016576; visual cylinder length=0.03000514686678052 radius=0.011167783570016576
- link f32: geometry collision cylinder length=0.0376423688804056 radius=0.011167783570016576; visual cylinder length=0.0376423688804056 radius=0.011167783570016576
Joints:
- joint f12_slot_joint: origin xyz=0.0 0.0 0.03000800623721414 rpy=0.0 0.0 0.0 -> xyz=0.0 0.0 0.03000514686678052 rpy=0.0 0.0 0.0
- joint f13_slot_joint: origin xyz=0.0 0.0 0.04188812936951982 rpy=0.0 0.0 0.0 -> xyz=0.0 0.0 0.0376423688804056 rpy=0.0 0.0 0.0
- joint f22_slot_joint: origin xyz=0.0 0.0 0.03000800623721414 rpy=0.0 0.0 0.0 -> xyz=0.0 0.0 0.03000514686678052 rpy=0.0 0.0 0.0
- joint f23_slot_joint: origin xyz=0.0 0.0 0.04188812936951982 rpy=0.0 0.0 0.0 -> xyz=0.0 0.0 0.0376423688804056 rpy=0.0 0.0 0.0
- joint f32_slot_joint: origin xyz=0.0 0.0 0.03000800623721414 rpy=0.0 0.0 0.0 -> xyz=0.0 0.0 0.03000514686678052 rpy=0.0 0.0 0.0
- joint f33_slot_joint: origin xyz=0.0 0.0 0.04188812936951982 rpy=0.0 0.0 0.0 -> xyz=0.0 0.0 0.0376423688804056 rpy=0.0 0.0 0.0

File: assets/gen_gripper/3f_2j/robot_3/model.urdf (robot description, URDF)
Before this commit: robot ur5_3f2j, 24 links, 23 joints
Links:
- link f11: geometry collision cylinder length=0.03952326522000266 radius=0.014078158525035238; visual cylinder length=0.03952326522000266 radius=0.014078158525035238
- link f12: geometry collision cylinder length=0.03087151310416337 radius=0.014078158525035238; visual cylinder length=0.03087151310416337 radius=0.014078158525035238
- link f21: geometry collision cylinder length=0.03952326522000266 radius=0.014078158525035238; visual cylinder length=0.03952326522000266 radius=0.014078158525035238
- link f22: geometry collision cylinder length=0.03087151310416337 radius=0.014078158525035238; visual cylinder length=0.03087151310416337 radius=0.014078158525035238
- link f31: geometry collision cylinder length=0.03952326522000266 radius=0.014078158525035238; visual cylinder length=0.03952326522000266 radius=0.014078158525035238
- link f32: geometry collision cylinder length=0.03087151310416337 radius=0.014078158525035238; visual cylinder length=0.03087151310416337 radius=0.014078158525035238
Joints:
- joint f12_slot_joint: origin xyz=0.0 0.0 0.044813968120004134 rpy=0.0 0.0 0.0 -> xyz=0.0 0.0 0.03952326522000266 rpy=0.0 0.0 0.0
- joint f13_slot_joint: origin xyz=0.0 0.0 0.031355687050920796 rpy=0.0 0.0 0.0 -> xyz=0.0 0.0 0.03087151310416337 rpy=0.0 0.0 0.0
- joint f22_slot_joint: origin xyz=0.0 0.0 0.044813968120004134 rpy=0.0 0.0 0.0 -> xyz=0.0 0.0 0.03952326522000266 rpy=0.0 0.0 0.0
- joint f23_slot_joint: origin xyz=0.0 0.0 0.031355687050920796 rpy=0.0 0.0 0.0 -> xyz=0.0 0.0 0.03087151310416337 rpy=0.0 0.0 0.0
- joint f32_slot_joint: origin xyz=0.0 0.0 0.044813968120004134 rpy=0.0 0.0 0.0 -> xyz=0.0 0.0 0.03952326522000266 rpy=0.0 0.0 0.0
- joint f33_slot_joint: origin xyz=0.0 0.0 0.031355687050920796 rpy=0.0 0.0 0.0 -> xyz=0.0 0.0 0.03087151310416337 rpy=0.0 0.0 0.0
